File: Eagle/LED-Schematic.sch (EAGLE design)
At the start: 8 parts, among them Q1 INFINEON_IRLB8721PBFINFINEON_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, Q2 INFINEON_IRLB8721PBFINFINEON_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, Q3 INFINEON_IRLB8721PBFINFINEON_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, X1 DG3XX-03-3.5, X2 DG3XX-03-3.5, X3 DG3XX-03-3.5, X4 DG3XX-03-3.5

Commit message: Integrated
Parts:
- removed X3: DG3XX-03-3.5, degson:DG3XX-03-3.5
- added R1, R2, R3: 10.0, SparkFun-Resistors:10OHM-1/4W-1%(PTH)
- added U1: HC-SR04, HC-SR04:HC-SR04
Connections:
- net 12V: now also X2-2.KL; no longer X3-3.KL
- net 5V: now also U1.VCC; no longer X3-1.KL
- net B-LED: now also R3.2
- net ECHO-SENSE: now also U1.ECHO; no longer X2-3.KL
- net G-LED: now also R2.2
- net GND: now also R1.1, R2.1, R3.1, U1.GND, X2-3.KL; no longer X3-2.KL, X4-1.KL
- net R-LED: now also R1.2
- net TRIG-SENSE: now also U1.TRIG; no longer X2-2.KL
Other:
- note added: "12V LED"
- note added: "LED Chanels"
- note removed: "LED OUT"
- note removed: "SENSOR"
- moved on the sheet: ARDUINO_NANO1, X1-1, X1-2, X1-3, X2-1, X2-2, X2-3, X4-1, X4-2, X4-3
